File: hardware/kicad/mojoback_sram.kicad_pcb (KiCad board)
At the start: 2 copper layers, 73 x 98.4 mm, 27 parts, among them U2 kl_bitsy

Commit message: who cares?
Other:
- net class Default removed
